Commit message: fix bug

File: pinky_description/urdf/robot_core.xacro (robot description, xacro)
@@ -41,5 +41,6 @@
             </geometry>
         </collision>
-        <xacro:inertial_box mass="${chassis_mass}" x="${chassis_length}" y="${chassis_width}" z="${chassis_height}">
+        <xacro:inertial_box mass="${chassis_mass}" x="${chassis_length}" y="${chassis_width}"
+                            z="${chassis_height}">
             <origin xyz="-0.01 0 0.01" rpy="0 0 0"/>
         </xacro:inertial_box>
@@ -51,5 +52,5 @@
     </joint>
 	<link name="caster">
-    <visual>
+        <visual>
             <origin xyz="0 0 0" rpy="0 0 0"/>
             <geometry>
